Commit message: Teleoperation working. Optimized meshes.

File: urdf/osr.urdf.xacro (robot description, xacro)
@@ -1,8 +1,14 @@
 <?xml version="1.0" encoding="utf-8"?>
 <!--
-    Title: Open Source Rover (OSR) Model
-    Description: This is the model that gets spawned when the launch file runs.
-    Version: v1.0, 03/2023
-    Tested with: ROS Noetic, Linux Ubuntu 20.04 LTS
+    Title:
+      Open Source Rover (OSR) Model
+    Description:
+      This is the model that gets spawned when the launch file runs.
+    Version:
+      v1.0, 03/2023
+    Tested with:
+      ROS Noetic, Linux Ubuntu 20.04 LTS
+    References:
+      Engineering Toolbox, https://www.engineeringtoolbox.com/friction-coefficients-d_778.html
 -->
 <robot
@@ -41,8 +47,8 @@
   <xacro:include filename="$(find osr)/urdf/osr_geometry.urdf.xacro" />
   <!-- **************** Wheel elements **************** -->
-  <!-- TODO: find real friction values -->
+  <!-- Rubber on dry asphalt (see reference) -->
   <gazebo reference="front_left_wheel">
-      <mu1 value="0.2"/>
-      <mu2 value="0.2"/>
+      <mu1 value="0.9"/>
+      <mu2 value="0.9"/>
       <kp value="10000000.0" />
       <kd value="1.0" />
@@ -50,6 +56,6 @@
   </gazebo>
   <gazebo reference="front_right_wheel">
-      <mu1 value="0.2"/>
-      <mu2 value="0.2"/>
+      <mu1 value="0.9"/>
+      <mu2 value="0.9"/>
       <kp value="10000000.0" />
       <kd value="1.0" />
@@ -57,6 +63,6 @@
   </gazebo>
   <gazebo reference="middle_left_wheel">
-      <mu1 value="0.2"/>
-      <mu2 value="0.2"/>
+      <mu1 value="0.9"/>
+      <mu2 value="0.9"/>
       <kp value="10000000.0" />
       <kd value="1.0" />
@@ -64,6 +70,6 @@
   </gazebo>
   <gazebo reference="middle_right_wheel">
-      <mu1 value="0.2"/>
-      <mu2 value="0.2"/>
+      <mu1 value="0.9"/>
+      <mu2 value="0.9"/>
       <kp value="10000000.0" />
       <kd value="1.0" />
@@ -71,6 +77,6 @@
   </gazebo>
   <gazebo reference="back_left_wheel">
-      <mu1 value="0.2"/>
-      <mu2 value="0.2"/>
+      <mu1 value="0.9"/>
+      <mu2 value="0.9"/>
       <kp value="10000000.0" />
       <kd value="1.0" />
@@ -78,6 +84,6 @@
   </gazebo>
   <gazebo reference="back_right_wheel">
-      <mu1 value="0.2"/>
-      <mu2 value="0.2"/>
+      <mu1 value="0.9"/>
+      <mu2 value="0.9"/>
       <kp value="10000000.0" />
       <kd value="1.0" />
@@ -85,5 +91,4 @@
   </gazebo>
   <!-- **************** Transmissions **************** -->
-  <!-- TODO: add transmissions for all moving joints or only for those with motors? -->
   <!-- Wheels -->
   <transmission name="front_left_wheel_trans">

File: urdf/osr_geometry.urdf.xacro (robot description, xacro)
@@ -1,8 +1,18 @@
 <?xml version="1.0" encoding="utf-8"?>
 <!--
-    Title: Open Source Rover (OSR) Model geometry
-    Description: This contains the geometry for the links and joints.
-    Version: v1.0, 03/2023
-    Tested with: ROS Noetic, Linux Ubuntu 20.04 LTS
+    Title:
+      Open Source Rover (OSR) Model geometry
+    Description:
+      This contains the geometry for the links and joints of the rover.
+      Meshes are from https://github.com/nasa-jpl/open-source-rover.
+    Version:
+      v1.0, 03/2023
+    Tested with:
+      ROS Noetic, Linux Ubuntu 20.04 LTS
+    References:
+      45 RPM HD Premium Planetary Gear Motor (datasheet),
+        https://www.servocity.com/content/downloads/45_rpm_hd_precision_planetary_gearmotor_-_specifications.pdf
+      5202 Series Yellow Jacket Planetary Gear Motor (datasheet),
+        https://www.gobilda.com/content/spec_sheets/5202-0002-0027_spec_sheet.pdf
 -->
 <!-- **************** Model geometry for OSR **************** -->
@@ -243,6 +253,6 @@
       lower="-0.7854"
       upper="0.7854"
-      effort="1000"
-      velocity="0" />
+      effort="2.0"
+      velocity="4.0" />
   </joint>
   <link
@@ -298,4 +308,7 @@
     <axis
       xyz="0 0 1" />
+    <limit
+      effort="3.5"
+      velocity="23"/>
   </joint>
   <link
@@ -351,4 +364,7 @@
     <axis
       xyz="0 0 1" />
+    <limit
+      effort="3.5"
+      velocity="23"/>
   </joint>
   <link
@@ -407,6 +423,6 @@
       lower="-0.7854"
       upper="0.7854"
-      effort="1000"
-      velocity="0" />
+      effort="2.0"
+      velocity="4.0" />
   </joint>
   <link
@@ -462,4 +478,7 @@
     <axis
       xyz="0 0 1" />
+    <limit
+      effort="3.5"
+      velocity="23"/>
   </joint>
   <link
@@ -634,6 +653,6 @@
       lower="-0.7854"
       upper="0.7854"
-      effort="1000"
-      velocity="0" />
+      effort="2.0"
+      velocity="4.0" />
   </joint>
   <link
@@ -689,4 +708,7 @@
     <axis
       xyz="0 0 1" />
+    <limit
+      effort="3.5"
+      velocity="23"/>
   </joint>
   <link
@@ -742,4 +764,7 @@
     <axis
       xyz="0 0 1" />
+    <limit
+      effort="3.5"
+      velocity="23"/>
   </joint>
   <link
@@ -798,6 +823,6 @@
       lower="-0.7854"
       upper="0.7854"
-      effort="1000"
-      velocity="0" />
+      effort="2.0"
+      velocity="4.0" />
   </joint>
   <link
@@ -853,4 +878,7 @@
     <axis
       xyz="0 0 1" />
+    <limit
+      effort="3.5"
+      velocity="23"/>
   </joint>
 </robot>

Commit message: Implemented joint limits as parameters

File: urdf/osr.urdf.xacro (robot description, xacro)
@@ -46,5 +46,5 @@
   <xacro:controller_plugin_gazebo />
   <!-- **************** Model geometry **************** -->
-  <xacro:include filename="$(find osr)/urdf/osr_geometry.urdf.xacro" />
+  <xacro:include filename="$(find osr)/urdf/osr_geometry.urdf.xacro"/>
   <!-- **************** Wheel elements **************** -->
   <!-- Rubber on dry asphalt (see reference) -->

File: urdf/osr_geometry.urdf.xacro (robot description, xacro)
@@ -12,8 +12,6 @@
       Linux Ubuntu, 20.04 LTS
     References:
-      45 RPM HD Premium Planetary Gear Motor (datasheet),
-        https://www.servocity.com/content/downloads/45_rpm_hd_precision_planetary_gearmotor_-_specifications.pdf
-      5202 Series Yellow Jacket Planetary Gear Motor (datasheet),
-        https://www.gobilda.com/content/spec_sheets/5202-0002-0027_spec_sheet.pdf
+      - corner-motor-datasheet (pdf)
+      - drive-motor-datasheet (pdf)
 -->
 <!-- **************** Model geometry for OSR **************** -->
@@ -21,4 +19,13 @@
   xmlns:xacro="http://ros.org/wiki/xacro"
   name="osr_geometry">
+  <!-- Load parameter values from parameter file -->
+  <xacro:property name="yaml_file" value="$(find osr)/config/osr_parameters.yaml" />
+  <xacro:property name="yaml_dict" value="${xacro.load_yaml(yaml_file)}"/>
+  <xacro:property name="steer_angle_max" value="${yaml_dict['steer_angle_max']}" />
+  <xacro:property name="steer_angle_min" value="${yaml_dict['steer_angle_min']}" />
+  <xacro:property name="steer_effort_max" value="${yaml_dict['steer_effort_max']}" />
+  <xacro:property name="steer_vel_max" value="${yaml_dict['steer_vel_max']}" />
+  <xacro:property name="drive_effort_max" value="${yaml_dict['drive_effort_max']}" />
+  <xacro:property name="drive_vel_max" value="${yaml_dict['drive_vel_max']}" />
   <link
     name="base_footprint">
@@ -252,8 +259,8 @@
       xyz="0 0 -0.999999999999988" />
     <limit
-      lower="-0.7854"
-      upper="0.7854"
-      effort="2.0"
-      velocity="4.0" />
+      lower="${steer_angle_min}"
+      upper="${steer_angle_max}"
+      effort="${steer_effort_max}"
+      velocity="${steer_vel_max}" />
   </joint>
   <link
@@ -310,6 +317,6 @@
       xyz="0 0 1" />
     <limit
-      effort="3.5"
-      velocity="23"/>
+      effort="${drive_effort_max}"
+      velocity="${drive_vel_max}"/>
   </joint>
   <link
@@ -366,6 +373,6 @@
       xyz="0 0 1" />
     <limit
-      effort="3.5"
-      velocity="23"/>
+      effort="${drive_effort_max}"
+      velocity="${drive_vel_max}"/>
   </joint>
   <link
@@ -422,8 +429,8 @@
       xyz="0 0 -1" />
     <limit
-      lower="-0.7854"
-      upper="0.7854"
-      effort="2.0"
-      velocity="4.0" />
+      lower="${steer_angle_min}"
+      upper="${steer_angle_max}"
+      effort="${steer_effort_max}"
+      velocity="${steer_vel_max}" />
   </joint>
   <link
@@ -480,6 +487,6 @@
       xyz="0 0 1" />
     <limit
-      effort="3.5"
-      velocity="23"/>
+      effort="${drive_effort_max}"
+      velocity="${drive_vel_max}"/>
   </joint>
   <link
@@ -652,8 +659,8 @@
       xyz="0 0 -1" />
     <limit
-      lower="-0.7854"
-      upper="0.7854"
-      effort="2.0"
-      velocity="4.0" />
+      lower="${steer_angle_min}"
+      upper="${steer_angle_max}"
+      effort="${steer_effort_max}"
+      velocity="${steer_vel_max}" />
   </joint>
   <link
@@ -710,6 +717,6 @@
       xyz="0 0 1" />
     <limit
-      effort="3.5"
-      velocity="23"/>
+      effort="${drive_effort_max}"
+      velocity="${drive_vel_max}"/>
   </joint>
   <link
@@ -766,6 +773,6 @@
       xyz="0 0 1" />
     <limit
-      effort="3.5"
-      velocity="23"/>
+      effort="${drive_effort_max}"
+      velocity="${drive_vel_max}"/>
   </joint>
   <link
@@ -822,8 +829,8 @@
       xyz="0 0 -1" />
     <limit
-      lower="-0.7854"
-      upper="0.7854"
-      effort="2.0"
-      velocity="4.0" />
+      lower="${steer_angle_min}"
+      upper="${steer_angle_max}"
+      effort="${steer_effort_max}"
+      velocity="${steer_vel_max}" />
   </joint>
   <link
@@ -880,6 +887,6 @@
       xyz="0 0 1" />
     <limit
-      effort="3.5"
-      velocity="23"/>
+      effort="${drive_effort_max}"
+      velocity="${drive_vel_max}"/>
   </joint>
 </robot>

Commit message: Added friction, stiffness and damping as parameters

File: urdf/osr.urdf.xacro (robot description, xacro)
@@ -16,5 +16,8 @@
   xmlns:xacro="http://ros.org/wiki/xacro"
   name="osr">
-  <!-- **************** Gazebo plugin for mimicing joints **************** -->
+  <!-- Load parameter values from parameter file -->
+  <xacro:property name="yaml_file" value="$(find osr)/config/osr_parameters.yaml" />
+  <xacro:property name="yaml_dict" value="${xacro.load_yaml(yaml_file)}"/>
+  <!--  Gazebo plugin for mimicing joints  -->
   <xacro:macro name="mimic_joint_plugin_gazebo" params="name_prefix parent_joint mimic_joint has_pid:=false multiplier:=1.0 offset:=0 sensitiveness:=0.0 max_effort:=1.0 robot_namespace:=''">
     <gazebo>
@@ -35,5 +38,5 @@
     </gazebo>
   </xacro:macro>
-  <!-- **************** Gazebo plugin for ROS control **************** -->
+  <!--  Gazebo plugin for ROS control  -->
   <!-- TODO: change to own namespace -->
   <xacro:macro name="controller_plugin_gazebo" params="robot_namespace:=''">
@@ -45,52 +48,55 @@
   </xacro:macro>
   <xacro:controller_plugin_gazebo />
-  <!-- **************** Model geometry **************** -->
+  <!--  Model geometry  -->
   <xacro:include filename="$(find osr)/urdf/osr_geometry.urdf.xacro"/>
-  <!-- **************** Wheel elements **************** -->
+  <!--  Wheel elements  -->
   <!-- Rubber on dry asphalt (see reference) -->
+  <xacro:property name="friction_1" value="${yaml_dict['friction_1']}" />
+  <xacro:property name="friction_2" value="${yaml_dict['friction_2']}" />
+  <xacro:property name="stiffness" value="${yaml_dict['stiffness']}" />
+  <xacro:property name="damping" value="${yaml_dict['damping']}" />
   <gazebo reference="front_left_wheel">
-      <mu1 value="0.9"/>
-      <mu2 value="0.9"/>
-      <kp value="10000000.0" />
-      <kd value="1.0" />
+      <mu1 value="${friction_1}"/>
+      <mu2 value="${friction_2}"/>
+      <kp value="${stiffness}" />
+      <kd value="${damping}" />
       <material>Gazebo/Grey</material>
   </gazebo>
   <gazebo reference="front_right_wheel">
-      <mu1 value="0.9"/>
-      <mu2 value="0.9"/>
-      <kp value="10000000.0" />
-      <kd value="1.0" />
+      <mu1 value="${friction_1}"/>
+      <mu2 value="${friction_2}"/>
+      <kp value="${stiffness}" />
+      <kd value="${damping}" />
       <material>Gazebo/Grey</material>
   </gazebo>
   <gazebo reference="middle_left_wheel">
-      <mu1 value="0.9"/>
-      <mu2 value="0.9"/>
-      <kp value="10000000.0" />
-      <kd value="1.0" />
+      <mu1 value="${friction_1}"/>
+      <mu2 value="${friction_2}"/>
+      <kp value="${stiffness}" />
+      <kd value="${damping}" />
       <material>Gazebo/Grey</material>
   </gazebo>
   <gazebo reference="middle_right_wheel">
-      <mu1 value="0.9"/>
-      <mu2 value="0.9"/>
-      <kp value="10000000.0" />
-      <kd value="1.0" />
+      <mu1 value="${friction_1}"/>
+      <mu2 value="${friction_2}"/>
+      <kp value="${stiffness}" />
+      <kd value="${damping}" />
       <material>Gazebo/Grey</material>
   </gazebo>
   <gazebo reference="back_left_wheel">
-      <mu1 value="0.9"/>
-      <mu2 value="0.9"/>
-      <kp value="10000000.0" />
-      <kd value="1.0" />
+      <mu1 value="${friction_1}"/>
+      <mu2 value="${friction_2}"/>
+      <kp value="${stiffness}" />
+      <kd value="${damping}" />
       <material>Gazebo/Grey</material>
   </gazebo>
   <gazebo reference="back_right_wheel">
-      <mu1 value="0.9"/>
-      <mu2 value="0.9"/>
-      <kp value="10000000.0" />
-      <kd value="1.0" />
+      <mu1 value="${friction_1}"/>
+      <mu2 value="${friction_2}"/>
+      <kp value="${stiffness}" />
+      <kd value="${damping}" />
       <material>Gazebo/Grey</material>
   </gazebo>
-  <!-- **************** Transmissions **************** -->
-  <!-- Wheels -->
+  <!-- Wheel transmissions -->
   <transmission name="front_left_wheel_trans">
     <type>transmission_interface/SimpleTransmission</type>
@@ -147,5 +153,5 @@
     </joint>
   </transmission>
-  <!-- Corner steering motors -->
+  <!-- Steering motor transmissions -->
   <transmission name="front_left_corner_trans">
     <type>transmission_interface/SimpleTransmission</type>

File: urdf/osr_geometry.urdf.xacro (robot description, xacro)
@@ -20,6 +20,4 @@
   name="osr_geometry">
   <!-- Load parameter values from parameter file -->
-  <xacro:property name="yaml_file" value="$(find osr)/config/osr_parameters.yaml" />
-  <xacro:property name="yaml_dict" value="${xacro.load_yaml(yaml_file)}"/>
   <xacro:property name="steer_angle_max" value="${yaml_dict['steer_angle_max']}" />
   <xacro:property name="steer_angle_min" value="${yaml_dict['steer_angle_min']}" />
