Commit message: Added rocker limits as parameters

File: urdf/osr_geometry.urdf.xacro (robot description, xacro)
@@ -26,4 +26,6 @@
   <xacro:property name="drive_effort_max" value="${yaml_dict['drive_effort_max']}" />
   <xacro:property name="drive_vel_max" value="${yaml_dict['drive_vel_max']}" />
+  <xacro:property name="rocker_limit_upper" value="${yaml_dict['rocker_limit_upper']}" />
+  <xacro:property name="rocker_limit_lower" value="${yaml_dict['rocker_limit_lower']}" />
   <link
     name="base_footprint">
@@ -137,6 +139,6 @@
       xyz="0 0 1" />
     <limit
-      lower="-0.1"
-      upper="0.1"
+      lower="${rocker_limit_lower}"
+      upper="${rocker_limit_upper}"
       effort="0"
       velocity="0" />
@@ -541,6 +543,6 @@
       xyz="0 0 1" />
     <limit
-      lower="-0.1"
-      upper="0.1"
+      lower="${rocker_limit_lower}"
+      upper="${rocker_limit_upper}"
       effort="0"
       velocity="0" />

Commit message: Updated the meshes to the new design

File: urdf/osr_geometry.urdf.xacro (robot description, xacro)
@@ -7,5 +7,5 @@
       Meshes are from https://github.com/nasa-jpl/open-source-rover.
     Version:
-      v1.0.0, 03/2023
+      v1.1.0, 04/2023
     Tested with:
       ROS Noetic
@@ -50,15 +50,15 @@
     <inertial>
       <origin
-        xyz="-0.16002 -0.00015951 -0.059815"
-        rpy="0 0 0" />
-      <mass
-        value="1.3874" />
-      <inertia
-        ixx="0.0060646"
-        ixy="3.4445E-11"
-        ixz="-3.7962E-09"
-        iyy="0.008315"
-        iyz="-3.0768E-05"
-        izz="0.013019" />
+        xyz="-0.14756 -6.6173E-06 -0.048928"
+        rpy="0 0 0" />
+      <mass
+        value="1.9413" />
+      <inertia
+        ixx="0.0077101"
+        ixy="2.0608E-08"
+        ixz="9.3168E-08"
+        iyy="0.011398"
+        iyz="-3.7258E-09"
+        izz="0.017109" />
     </inertial>
     <visual>
@@ -90,14 +90,14 @@
     <inertial>
       <origin
-        xyz="-0.081315 0.0093907 -0.033982"
+        xyz="0.0093907 -0.081315 0.033982"
         rpy="0 0 0" />
       <mass
         value="0.54518" />
       <inertia
-        ixx="0.00030463"
+        ixx="0.00071766"
         ixy="-5.98E-05"
-        ixz="-7.683E-08"
-        iyy="0.00071766"
-        iyz="-8.8606E-07"
+        ixz="8.8606E-07"
+        iyy="0.00030463"
+        iyz="7.6825E-08"
         izz="0.0008578" />
     </inertial>
@@ -130,6 +130,6 @@
     type="revolute">
     <origin
-      xyz="-0.173744384181607 0.190500000000003 -0.0594359999999901"
-      rpy="-1.57079632679489 0 0" />
+      xyz="-0.173736 0.190375827761485 -0.0594359999999915"
+      rpy="1.57079632679488 1.5707963267949 0" />
     <parent
       link="base_link" />
@@ -137,8 +137,8 @@
       link="left_rocker" />
     <axis
-      xyz="0 0 1" />
-    <limit
-      lower="${rocker_limit_lower}"
-      upper="${rocker_limit_upper}"
+      xyz="0 0 -1" />
+    <limit
+      lower="-0.1"
+      upper="0.1"
       effort="0"
       velocity="0" />
@@ -152,5 +152,5 @@
     <inertial>
       <origin
-        xyz="0.11235 -0.038605 0.3532"
+        xyz="0.11231 -0.038529 0.35308"
         rpy="0 0 0" />
       <mass
@@ -159,7 +159,7 @@
         ixx="0.0003158"
         ixy="7.6325E-05"
-        ixz="3.8116E-08"
+        ixz="3.8124E-08"
         iyy="0.00032094"
-        iyz="8.1411E-07"
+        iyz="8.1409E-07"
         izz="0.00046244" />
     </inertial>
@@ -192,6 +192,6 @@
     type="continuous">
     <origin
-      xyz="0.187139225679552 0.102147968996281 -0.38522275000001"
-      rpy="0 0 0" />
+      xyz="0.102072501603827 0.187180386097456 0.38509857776149"
+      rpy="-3.14159263778426 0 1.57079617385391" />
     <parent
       link="left_rocker" />
@@ -199,5 +199,5 @@
       link="left_bogie" />
     <axis
-      xyz="0 0 -0.999999999999994" />
+      xyz="0 0 -1" />
     <limit
       lower="0"
@@ -250,6 +250,6 @@
     type="revolute">
     <origin
-      xyz="0.215421536981298 0.00545134107835665 0.351039494185675"
-      rpy="1.57079621520304 0 0" />
+      xyz="0.215380376567892 0.00552677512849714 0.350915322468129"
+      rpy="1.57079631098936 0 0" />
     <parent
       link="left_bogie" />
@@ -268,15 +268,15 @@
     <inertial>
       <origin
-        xyz="-8.2916E-07 -1.7142E-07 0.00092227"
-        rpy="0 0 0" />
-      <mass
-        value="1.4215" />
-      <inertia
-        ixx="0.0038879"
-        ixy="9.182E-08"
-        ixz="1.0732E-07"
-        iyy="0.003888"
-        iyz="-7.856E-08"
-        izz="0.0058222" />
+        xyz="4.9366E-10 -1.3882E-10 0.0071368"
+        rpy="0 0 0" />
+      <mass
+        value="0.61431" />
+      <inertia
+        ixx="0.0011197"
+        ixy="5.7673E-08"
+        ixz="-3.3832E-16"
+        iyy="0.0011199"
+        iyz="5.6789E-17"
+        izz="0.001892" />
     </inertial>
     <visual>
@@ -291,5 +291,5 @@
         name="">
         <color
-          rgba="0.29412 0.29412 0.29412 1" />
+          rgba="0.62745 0.62745 0.62745 1" />
       </material>
     </visual>
@@ -308,6 +308,6 @@
     type="continuous">
     <origin
-      xyz="-0.00017181 -4.3245E-05 -0.12889"
-      rpy="-1.5708 0 0" />
+      xyz="-0.00017180884072221 -4.3244793997782E-05 -0.128892240205177"
+      rpy="-1.57079632679486 0 0" />
     <parent
       link="front_left_corner" />
@@ -318,5 +318,5 @@
     <limit
       effort="${drive_effort_max}"
-      velocity="${drive_vel_max}"/>
+      velocity="${drive_vel_max}" />
   </joint>
   <link
@@ -324,15 +324,15 @@
     <inertial>
       <origin
-        xyz="-8.2252E-07 -2.0291E-07 0.00092227"
-        rpy="0 0 0" />
-      <mass
-        value="1.4215" />
-      <inertia
-        ixx="0.0038879"
-        ixy="8.7004E-08"
-        ixz="1.1027E-07"
-        iyy="0.003888"
-        iyz="-7.439E-08"
-        izz="0.0058222" />
+        xyz="4.4851E-10 2.7786E-10 0.0071368"
+        rpy="0 0 0" />
+      <mass
+        value="0.61431" />
+      <inertia
+        ixx="0.0011197"
+        ixy="5.2219E-08"
+        ixz="-1.5331E-16"
+        iyy="0.0011199"
+        iyz="-3.1316E-17"
+        izz="0.001892" />
     </inertial>
     <visual>
@@ -347,5 +347,5 @@
         name="">
         <color
-          rgba="0.29412 0.29412 0.29412 1" />
+          rgba="0.62745 0.62745 0.62745 1" />
       </material>
     </visual>
@@ -364,5 +364,5 @@
     type="continuous">
     <origin
-      xyz="-0.063913345312238 0.103041664281169 0.436572914004881"
+      xyz="-0.0639545058516444 0.103117089777728 0.436448751635148"
       rpy="0 0 0" />
     <parent
@@ -374,5 +374,5 @@
     <limit
       effort="${drive_effort_max}"
-      velocity="${drive_vel_max}"/>
+      velocity="${drive_vel_max}" />
   </joint>
   <link
@@ -420,6 +420,6 @@
     type="revolute">
     <origin
-      xyz="-0.186901909356396 0.0959973702109308 -0.0342697447940019"
-      rpy="1.57079632679489 0 -0.0409113907910423" />
+      xyz="0.095997370210931 -0.186901909356396 0.0342697447940012"
+      rpy="-1.5707963267949 0 1.61170771758594" />
     <parent
       link="left_rocker" />
@@ -438,15 +438,15 @@
     <inertial>
       <origin
-        xyz="-8.2953E-07 -1.7315E-07 0.00092227"
-        rpy="0 0 0" />
-      <mass
-        value="1.4215" />
-      <inertia
-        ixx="0.0038879"
-        ixy="9.1817E-08"
-        ixz="1.0732E-07"
-        iyy="0.003888"
-        iyz="-7.8477E-08"
-        izz="0.0058222" />
+        xyz="4.3795E-10 6.9914E-10 0.0071368"
+        rpy="0 0 0" />
+      <mass
+        value="0.61431" />
+      <inertia
+        ixx="0.0011197"
+        ixy="5.7673E-08"
+        ixz="-1.2405E-16"
+        iyy="0.0011199"
+        iyz="1.2035E-16"
+        izz="0.001892" />
     </inertial>
     <visual>
@@ -461,5 +461,5 @@
         name="">
         <color
-          rgba="0.29412 0.29412 0.29412 1" />
+          rgba="0.62745 0.62745 0.62745 1" />
       </material>
     </visual>
@@ -478,6 +478,6 @@
     type="continuous">
     <origin
-      xyz="0.00017181 4.3245E-05 -0.12889"
-      rpy="-1.5708 0 0" />
+      xyz="0.000171808840937315 4.32447939933134E-05 -0.128892240205023"
+      rpy="-1.57079632679486 0 0" />
     <parent
       link="back_left_corner" />
@@ -488,5 +488,5 @@
     <limit
       effort="${drive_effort_max}"
-      velocity="${drive_vel_max}"/>
+      velocity="${drive_vel_max}" />
   </joint>
   <link
@@ -494,14 +494,14 @@
     <inertial>
       <origin
-        xyz="-0.081411 0.0085199 0.034486"
+        xyz="-0.081408 0.0085528 0.03461"
         rpy="0 0 0" />
       <mass
         value="0.54518" />
       <inertia
-        ixx="0.00030593"
-        ixy="-6.4225E-05"
-        ixz="-6.7388E-08"
-        iyy="0.00071636"
-        iyz="-8.868E-07"
+        ixx="0.00030587"
+        ixy="-6.406E-05"
+        ixz="-6.7746E-08"
+        iyy="0.00071641"
+        iyz="-8.8677E-07"
         izz="0.0008578" />
     </inertial>
@@ -534,6 +534,6 @@
     type="revolute">
     <origin
-      xyz="-0.17374 -0.1905 -0.059436"
-      rpy="-1.5708 0 0" />
+      xyz="-0.173736 -0.190624172238515 -0.0594359999999888"
+      rpy="-1.5707963267949 0 0" />
     <parent
       link="base_link" />
@@ -543,6 +543,6 @@
       xyz="0 0 1" />
     <limit
-      lower="${rocker_limit_lower}"
-      upper="${rocker_limit_upper}"
+      lower="-0.1"
+      upper="0.1"
       effort="0"
       velocity="0" />
@@ -552,5 +552,5 @@
     <inertial>
       <origin
-        xyz="0.10915 -0.034095 -0.35298"
+        xyz="0.10919 -0.034171 -0.35286"
         rpy="0 0 0" />
       <mass
@@ -559,7 +559,7 @@
         ixx="0.00031636"
         ixy="7.664E-05"
-        ixz="3.8372E-08"
+        ixz="3.8142E-08"
         iyy="0.00032122"
-        iyz="9.6233E-07"
+        iyz="9.6276E-07"
         izz="0.00046272" />
     </inertial>
@@ -592,5 +592,5 @@
     type="continuous">
     <origin
-      xyz="0.188216644575796 0.100148826719136 0.384524249999983"
+      xyz="0.188216650413261 0.100148831558874 0.384524249999976"
       rpy="0 0 0" />
     <parent
@@ -599,5 +599,5 @@
       link="right_bogie" />
     <axis
-      xyz="0 0 -0.999999999994781" />
+      xyz="0 0 -0.999999999999974" />
     <limit
       lower="0"
@@ -650,6 +650,6 @@
     type="revolute">
     <origin
-      xyz="0.213266684003467 0.00945072449948589 -0.350254474673649"
-      rpy="1.57079955767686 0 0" />
+      xyz="0.213307849599925 0.00937420353549007 -0.350130330857906"
+      rpy="1.57079655183463 0 0" />
     <parent
       link="right_bogie" />
@@ -668,15 +668,15 @@
     <inertial>
       <origin
-        xyz="8.296E-07 -1.7167E-07 -0.00092227"
-        rpy="0 0 0" />
-      <mass
-        value="1.4215" />
-      <inertia
-        ixx="0.0038879"
-        ixy="-9.1827E-08"
-        ixz="1.0729E-07"
-        iyy="0.003888"
-        iyz="7.8574E-08"
-        izz="0.0058222" />
+        xyz="5.237E-11 -5.0691E-11 -0.0071368"
+        rpy="0 0 0" />
+      <mass
+        value="0.61431" />
+      <inertia
+        ixx="0.0011197"
+        ixy="-5.7673E-08"
+        ixz="-1.312E-16"
+        iyy="0.0011199"
+        iyz="-5.7322E-17"
+        izz="0.001892" />
     </inertial>
     <visual>
@@ -691,5 +691,5 @@
         name="">
         <color
-          rgba="0.29412 0.29412 0.29412 1" />
+          rgba="0.62745 0.62745 0.62745 1" />
       </material>
     </visual>
@@ -708,5 +708,5 @@
     type="continuous">
     <origin
-      xyz="-0.000171808840734172 -4.32447939935077E-05 -0.128892240205189"
+      xyz="-0.000171808840730647 -4.32447939935632E-05 -0.128892240205185"
       rpy="-1.57079632679494 0 0" />
     <parent
@@ -718,5 +718,5 @@
     <limit
       effort="${drive_effort_max}"
-      velocity="${drive_vel_max}"/>
+      velocity="${drive_vel_max}" />
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