Commit message: Renamed OSR to OSLR

File: urdf/oslr.urdf.xacro (robot description, xacro)
@@ -2,5 +2,5 @@
 <!--
     Title:
-      Open Source Rover (OSR) Model
+      Open Source Lunar Rover (oslr) Model
     Description:
       This is the model that gets spawned when the launch file runs.
@@ -15,7 +15,7 @@
 <robot
   xmlns:xacro="http://ros.org/wiki/xacro"
-  name="osr">
+  name="oslr">
   <!-- Load parameter values from parameter file -->
-  <xacro:property name="yaml_file" value="$(find osr)/config/osr_parameters.yaml" />
+  <xacro:property name="yaml_file" value="$(find oslr)/config/oslr_parameters.yaml" />
   <xacro:property name="yaml_dict" value="${xacro.load_yaml(yaml_file)}"/>
   <!--  Gazebo plugin for mimicing joints  -->
@@ -49,5 +49,5 @@
   <xacro:controller_plugin_gazebo />
   <!--  Model geometry  -->
-  <xacro:include filename="$(find osr)/urdf/osr_geometry.urdf.xacro"/>
+  <xacro:include filename="$(find oslr)/urdf/oslr_geometry.urdf.xacro"/>
   <!--  Wheel elements  -->
   <!-- Rubber on dry asphalt (see reference) -->

File: urdf/oslr_geometry.urdf.xacro (robot description, xacro)
@@ -2,5 +2,5 @@
 <!--
     Title:
-      Open Source Rover (OSR) Model geometry
+      Open Source Lunar Rover (oslr) Model geometry
     Description:
       This contains the geometry for the links and joints of the rover.
@@ -15,8 +15,8 @@
       - drive-motor-datasheet (pdf)
 -->
-<!-- **************** Model geometry for OSR **************** -->
+<!-- **************** Model geometry for oslr **************** -->
 <robot
   xmlns:xacro="http://ros.org/wiki/xacro"
-  name="osr_geometry">
+  name="oslr_geometry">
   <!-- Load parameter values from parameter file -->
   <xacro:property name="steer_angle_max" value="${yaml_dict['steer_angle_max']}" />
@@ -68,5 +68,5 @@
       <geometry>
         <mesh
-          filename="package://osr/meshes/base_link.STL" />
+          filename="package://oslr/meshes/base_link.STL" />
       </geometry>
       <material
@@ -82,5 +82,5 @@
       <geometry>
         <mesh
-          filename="package://osr/meshes/base_link.STL" />
+          filename="package://oslr/meshes/base_link.STL" />
       </geometry>
     </collision>
@@ -108,5 +108,5 @@
       <geometry>
         <mesh
-          filename="package://osr/meshes/left_rocker.STL" />
+          filename="package://oslr/meshes/left_rocker.STL" />
       </geometry>
       <material
@@ -122,5 +122,5 @@
       <geometry>
         <mesh
-          filename="package://osr/meshes/left_rocker.STL" />
+          filename="package://oslr/meshes/left_rocker.STL" />
       </geometry>
     </collision>
@@ -170,5 +170,5 @@
       <geometry>
         <mesh
-          filename="package://osr/meshes/left_bogie.STL" />
+          filename="package://oslr/meshes/left_bogie.STL" />
       </geometry>
       <material
@@ -184,5 +184,5 @@
       <geometry>
         <mesh
-          filename="package://osr/meshes/left_bogie.STL" />
+          filename="package://oslr/meshes/left_bogie.STL" />
       </geometry>
     </collision>
@@ -228,5 +228,5 @@
       <geometry>
         <mesh
-          filename="package://osr/meshes/front_left_corner.STL" />
+          filename="package://oslr/meshes/front_left_corner.STL" />
       </geometry>
       <material
@@ -242,5 +242,5 @@
       <geometry>
         <mesh
-          filename="package://osr/meshes/front_left_corner.STL" />
+          filename="package://oslr/meshes/front_left_corner.STL" />
       </geometry>
     </collision>
@@ -286,5 +286,5 @@
       <geometry>
         <mesh
-          filename="package://osr/meshes/front_left_wheel.STL" />
+          filename="package://oslr/meshes/front_left_wheel.STL" />
       </geometry>
       <material
@@ -300,5 +300,5 @@
       <geometry>
         <mesh
-          filename="package://osr/meshes/front_left_wheel.STL" />
+          filename="package://oslr/meshes/front_left_wheel.STL" />
       </geometry>
     </collision>
@@ -342,5 +342,5 @@
       <geometry>
         <mesh
-          filename="package://osr/meshes/middle_left_wheel.STL" />
+          filename="package://oslr/meshes/middle_left_wheel.STL" />
       </geometry>
       <material
@@ -356,5 +356,5 @@
       <geometry>
         <mesh
-          filename="package://osr/meshes/middle_left_wheel.STL" />
+          filename="package://oslr/meshes/middle_left_wheel.STL" />
       </geometry>
     </collision>
@@ -398,5 +398,5 @@
       <geometry>
         <mesh
-          filename="package://osr/meshes/back_left_corner.STL" />
+          filename="package://oslr/meshes/back_left_corner.STL" />
       </geometry>
       <material
@@ -412,5 +412,5 @@
       <geometry>
         <mesh
-          filename="package://osr/meshes/back_left_corner.STL" />
+          filename="package://oslr/meshes/back_left_corner.STL" />
       </geometry>
     </collision>
@@ -456,5 +456,5 @@
       <geometry>
         <mesh
-          filename="package://osr/meshes/back_left_wheel.STL" />
+          filename="package://oslr/meshes/back_left_wheel.STL" />
       </geometry>
       <material
@@ -470,5 +470,5 @@
       <geometry>
         <mesh
-          filename="package://osr/meshes/back_left_wheel.STL" />
+          filename="package://oslr/meshes/back_left_wheel.STL" />
       </geometry>
     </collision>
@@ -512,5 +512,5 @@
       <geometry>
         <mesh
-          filename="package://osr/meshes/right_rocker.STL" />
+          filename="package://oslr/meshes/right_rocker.STL" />
       </geometry>
       <material
@@ -526,5 +526,5 @@
       <geometry>
         <mesh
-          filename="package://osr/meshes/right_rocker.STL" />
+          filename="package://oslr/meshes/right_rocker.STL" />
       </geometry>
     </collision>
@@ -570,5 +570,5 @@
       <geometry>
         <mesh
-          filename="package://osr/meshes/right_bogie.STL" />
+          filename="package://oslr/meshes/right_bogie.STL" />
       </geometry>
       <material
@@ -584,5 +584,5 @@
       <geometry>
         <mesh
-          filename="package://osr/meshes/right_bogie.STL" />
+          filename="package://oslr/meshes/right_bogie.STL" />
       </geometry>
     </collision>
@@ -628,5 +628,5 @@
       <geometry>
         <mesh
-          filename="package://osr/meshes/front_right_corner.STL" />
+          filename="package://oslr/meshes/front_right_corner.STL" />
       </geometry>
       <material
@@ -642,5 +642,5 @@
       <geometry>
         <mesh
-          filename="package://osr/meshes/front_right_corner.STL" />
+          filename="package://oslr/meshes/front_right_corner.STL" />
       </geometry>
     </collision>
@@ -686,5 +686,5 @@
       <geometry>
         <mesh
-          filename="package://osr/meshes/front_right_wheel.STL" />
+          filename="package://oslr/meshes/front_right_wheel.STL" />
       </geometry>
       <material
@@ -700,5 +700,5 @@
       <geometry>
         <mesh
-          filename="package://osr/meshes/front_right_wheel.STL" />
+          filename="package://oslr/meshes/front_right_wheel.STL" />
       </geometry>
     </collision>
@@ -742,5 +742,5 @@
       <geometry>
         <mesh
-          filename="package://osr/meshes/middle_right_wheel.STL" />
+          filename="package://oslr/meshes/middle_right_wheel.STL" />
       </geometry>
       <material
@@ -756,5 +756,5 @@
       <geometry>
         <mesh
-          filename="package://osr/meshes/middle_right_wheel.STL" />
+          filename="package://oslr/meshes/middle_right_wheel.STL" />
       </geometry>
     </collision>
@@ -798,5 +798,5 @@
       <geometry>
         <mesh
-          filename="package://osr/meshes/back_right_corner.STL" />
+          filename="package://oslr/meshes/back_right_corner.STL" />
       </geometry>
       <material
@@ -812,5 +812,5 @@
       <geometry>
         <mesh
-          filename="package://osr/meshes/back_right_corner.STL" />
+          filename="package://oslr/meshes/back_right_corner.STL" />
       </geometry>
     </collision>
@@ -856,5 +856,5 @@
       <geometry>
         <mesh
-          filename="package://osr/meshes/back_right_wheel.STL" />
+          filename="package://oslr/meshes/back_right_wheel.STL" />
       </geometry>
       <material
@@ -870,5 +870,5 @@
       <geometry>
         <mesh
-          filename="package://osr/meshes/back_right_wheel.STL" />
+          filename="package://oslr/meshes/back_right_wheel.STL" />
       </geometry>
     </collision>
@@ -912,5 +912,5 @@
       <geometry>
         <mesh
-          filename="package://osr/meshes/navcam_vertical.STL" />
+          filename="package://oslr/meshes/navcam_vertical.STL" />
       </geometry>
       <material
@@ -926,5 +926,5 @@
       <geometry>
         <mesh
-          filename="package://osr/meshes/navcam_vertical.STL" />
+          filename="package://oslr/meshes/navcam_vertical.STL" />
       </geometry>
     </collision>
@@ -965,5 +965,5 @@
       <geometry>
         <mesh
-          filename="package://osr/meshes/navcam_horiz.STL" />
+          filename="package://oslr/meshes/navcam_horiz.STL" />
       </geometry>
       <material
@@ -979,5 +979,5 @@
       <geometry>
         <mesh
-          filename="package://osr/meshes/navcam_horiz.STL" />
+          filename="package://oslr/meshes/navcam_horiz.STL" />
       </geometry>
     </collision>

Commit message: Separated the OSLR model into components

File: urdf/oslr.urdf.xacro (robot description, xacro)
@@ -1,43 +1,41 @@
 <?xml version="1.0" encoding="utf-8"?>
 <!--
-    Title:
-      Open Source Lunar Rover (oslr) Model
-    Description:
-      This is the model that gets spawned when the launch file runs.
-    Version:
-      v1.0.0, 03/2023
-    Tested with:
-      ROS Noetic
-      Linux Ubuntu, 20.04 LTS
-    References:
-      Engineering Toolbox, https://www.engineeringtoolbox.com/friction-coefficients-d_778.html
+#
+# Title:
+#  Open Source Lunar Rover (OSLR) Model
+#
+# Author(s):
+#   andyjak
+#
+# Version:
+#   0.0.1, 08/2023
+#
+# Purpose:
+#   Main model of OSLR.
+#
+# Notes:
+#   Include this file in the launch file in order to spawn it.
+#
+# Test setup:
+#   - ROS Noetic
+#   - Ubuntu, 20.04 LTS
+#   - Python 3.8.10
+#
+# References:
+#   ...
+#
 -->
 <robot
   xmlns:xacro="http://ros.org/wiki/xacro"
   name="oslr">
-  <!-- Load parameter values from parameter file -->
+  <!-- Load parameter values from file (only needs to be done once) -->
   <xacro:property name="yaml_file" value="$(find oslr)/config/oslr_parameters.yaml" />
   <xacro:property name="yaml_dict" value="${xacro.load_yaml(yaml_file)}"/>
-  <!--  Gazebo plugin for mimicing joints  -->
-  <xacro:macro name="mimic_joint_plugin_gazebo" params="name_prefix parent_joint mimic_joint has_pid:=false multiplier:=1.0 offset:=0 sensitiveness:=0.0 max_effort:=1.0 robot_namespace:=''">
-    <gazebo>
-      <plugin name="${name_prefix}mimic_joint_plugin" filename="libroboticsgroup_gazebo_mimic_joint_plugin.so">
-        <joint>${parent_joint}</joint>
-        <mimicJoint>${mimic_joint}</mimicJoint>
-        <xacro:if value="${has_pid}">                     <!-- if set to true, PID parameters from "/gazebo_ros_control/pid_gains/${mimic_joint}" are loaded -->
-          <hasPID />
-        </xacro:if>
-        <multiplier>${multiplier}</multiplier>
-        <offset>${offset}</offset>
-        <sensitiveness>${sensitiveness}</sensitiveness>   <!-- if absolute difference between setpoint and process value is below this threshold, do nothing; 0.0 = disable [rad] -->
-        <maxEffort>${max_effort}</maxEffort>              <!-- only taken into account if has_pid:=true [Nm] -->
-        <xacro:unless value="${robot_namespace == ''}">
-          <robotNamespace>${robot_namespace}</robotNamespace>
-        </xacro:unless>
-      </plugin>
-    </gazebo>
-  </xacro:macro>
-  <!--  Gazebo plugin for ROS control  -->
-  <!-- TODO: change to own namespace -->
+  <!-- Load rover model components -->
+  <xacro:include filename="$(find oslr)/urdf/oslr_base.xacro"/>
+  <xacro:include filename="$(find oslr)/urdf/oslr_rockerbogie.xacro"/>
+  <xacro:include filename="$(find oslr)/urdf/oslr_wheels.xacro"/>
+  <xacro:include filename="$(find oslr)/urdf/oslr_navcam.xacro"/>
+  <!-- Load Gazebo plugin for ROS control -->
   <xacro:macro name="controller_plugin_gazebo" params="robot_namespace:=''">
     <gazebo>
@@ -48,145 +46,3 @@
   </xacro:macro>
   <xacro:controller_plugin_gazebo />
-  <!--  Model geometry  -->
-  <xacro:include filename="$(find oslr)/urdf/oslr_geometry.urdf.xacro"/>
-  <!--  Wheel elements  -->
-  <!-- Rubber on dry asphalt (see reference) -->
-  <xacro:property name="friction_1" value="${yaml_dict['friction_1']}" />
-  <xacro:property name="friction_2" value="${yaml_dict['friction_2']}" />
-  <xacro:property name="stiffness" value="${yaml_dict['stiffness']}" />
-  <xacro:property name="damping" value="${yaml_dict['damping']}" />
-  <gazebo reference="front_left_wheel">
-      <mu1 value="${friction_1}"/>
-      <mu2 value="${friction_2}"/>
-      <kp value="${stiffness}" />
-      <kd value="${damping}" />
-      <material>Gazebo/Grey</material>
-  </gazebo>
-  <gazebo reference="front_right_wheel">
-      <mu1 value="${friction_1}"/>
-      <mu2 value="${friction_2}"/>
-      <kp value="${stiffness}" />
-      <kd value="${damping}" />
-      <material>Gazebo/Grey</material>
-  </gazebo>
-  <gazebo reference="middle_left_wheel">
-      <mu1 value="${friction_1}"/>
-      <mu2 value="${friction_2}"/>
-      <kp value="${stiffness}" />
-      <kd value="${damping}" />
-      <material>Gazebo/Grey</material>
-  </gazebo>
-  <gazebo reference="middle_right_wheel">
-      <mu1 value="${friction_1}"/>
-      <mu2 value="${friction_2}"/>
-      <kp value="${stiffness}" />
-      <kd value="${damping}" />
-      <material>Gazebo/Grey</material>
-  </gazebo>
-  <gazebo reference="back_left_wheel">
-      <mu1 value="${friction_1}"/>
-      <mu2 value="${friction_2}"/>
-      <kp value="${stiffness}" />
-      <kd value="${damping}" />
-      <material>Gazebo/Grey</material>
-  </gazebo>
-  <gazebo reference="back_right_wheel">
-      <mu1 value="${friction_1}"/>
-      <mu2 value="${friction_2}"/>
-      <kp value="${stiffness}" />
-      <kd value="${damping}" />
-      <material>Gazebo/Grey</material>
-  </gazebo>
-  <!-- Wheel transmissions -->
-  <transmission name="front_left_wheel_trans">
-    <type>transmission_interface/SimpleTransmission</type>
-    <actuator name="front_left_wheel_motor">
-      <mechanicalReduction>1</mechanicalReduction>
-    </actuator>
-    <joint name="front_left_drive_joint">
-      <hardwareInterface>hardware_interface/EffortJointInterface</hardwareInterface>
-    </joint>
-  </transmission>
-  <transmission name="front_right_wheel_trans">
-    <type>transmission_interface/SimpleTransmission</type>
-    <actuator name="front_right_wheel_motor">
-      <mechanicalReduction>1</mechanicalReduction>
-    </actuator>
-    <joint name="front_right_drive_joint">
-      <hardwareInterface>hardware_interface/EffortJointInterface</hardwareInterface>
-    </joint>
-  </transmission>
-  <transmission name="middle_left_wheel_trans">
-    <type>transmission_interface/SimpleTransmission</type>
-    <actuator name="middle_left_wheel_motor">
-      <mechanicalReduction>1</mechanicalReduction>
-    </actuator>
-    <joint name="middle_left_drive_joint">
-      <hardwareInterface>hardware_interface/EffortJointInterface</hardwareInterface>
-    </joint>
-  </transmission>
-  <transmission name="middle_right_wheel_trans">
-    <type>transmission_interface/SimpleTransmission</type>
-    <actuator name="middle_right_wheel_motor">
-      <mechanicalReduction>1</mechanicalReduction>
-    </actuator>
-    <joint name="middle_right_drive_joint">
-      <hardwareInterface>hardware_interface/EffortJointInterface</hardwareInterface>
-    </joint>
-  </transmission>
-  <transmission name="back_left_wheel_trans">
-    <type>transmission_interface/SimpleTransmission</type>
-    <actuator name="back_left_wheel_motor">
-      <mechanicalReduction>1</mechanicalReduction>
-    </actuator>
-    <joint name="back_left_drive_joint">
-      <hardwareInterface>hardware_interface/EffortJointInterface</hardwareInterface>
-    </joint>
-  </transmission>
-  <transmission name="back_right_wheel_trans">
-    <type>transmission_interface/SimpleTransmission</type>
-    <actuator name="back_right_wheel_motor">
-      <mechanicalReduction>1</mechanicalReduction>
-    </actuator>
-    <joint name="back_right_drive_joint">
-      <hardwareInterface>hardware_interface/EffortJointInterface</hardwareInterface>
-    </joint>
-  </transmission>
-  <!-- Steering motor transmissions -->
-  <transmission name="front_left_corner_trans">
-    <type>transmission_interface/SimpleTransmission</type>
-    <actuator name="front_left_corner_motor">
-      <mechanicalReduction>1</mechanicalReduction>
-    </actuator>
-    <joint name="front_left_corner_joint">
-      <hardwareInterface>hardware_interface/EffortJointInterface</hardwareInterface>
-    </joint>
-  </transmission>
-  <transmission name="front_right_corner_trans">
-    <type>transmission_interface/SimpleTransmission</type>
-    <actuator name="front_right_corner_motor">
-      <mechanicalReduction>1</mechanicalReduction>
-    </actuator>
-    <joint name="front_right_corner_joint">
-      <hardwareInterface>hardware_interface/EffortJointInterface</hardwareInterface>
-    </joint>
-  </transmission>
-  <transmission name="back_left_corner_trans">
-    <type>transmission_interface/SimpleTransmission</type>
-    <actuator name="back_left_corner_motor">
-      <mechanicalReduction>1</mechanicalReduction>
-    </actuator>
-    <joint name="back_left_corner_joint">
-      <hardwareInterface>hardware_interface/EffortJointInterface</hardwareInterface>
-    </joint>
-  </transmission>
-  <transmission name="back_right_corner_trans">
-    <type>transmission_interface/SimpleTransmission</type>
-    <actuator name="back_right_corner_motor">
-      <mechanicalReduction>1</mechanicalReduction>
-    </actuator>
-    <joint name="back_right_corner_joint">
-      <hardwareInterface>hardware_interface/EffortJointInterface</hardwareInterface>
-    </joint>
-  </transmission>
 </robot>
