Commit message: Re-organized package structure into ROS standard

File: oslr_description/urdf/oslr.urdf.xacro (robot description, xacro)
@@ -15,5 +15,5 @@
 #
 # Notes:
-#   Include this file in the launch file in order to spawn it.
+#   Include this file in the launch file in order to spawn the model.
 #
 # Test setup:
@@ -23,5 +23,6 @@
 #
 # References:
-#   ...
+#   References are listed in the README.
+#   Comments that include a [number] refers to the index in the reference list.
 #
 -->
@@ -30,11 +31,11 @@
   name="oslr">
   <!-- Load parameter values from file (only needs to be done once) -->
-  <xacro:property name="yaml_file" value="$(find oslr)/config/oslr_parameters.yaml" />
+  <xacro:property name="yaml_file" value="$(find oslr_config)/config/oslr_parameters.yaml" />
   <xacro:property name="yaml_dict" value="${xacro.load_yaml(yaml_file)}"/>
   <!-- Load rover model components -->
-  <xacro:include filename="$(find oslr)/urdf/oslr_base.xacro"/>
-  <xacro:include filename="$(find oslr)/urdf/oslr_rockerbogie.xacro"/>
-  <xacro:include filename="$(find oslr)/urdf/oslr_wheels.xacro"/>
-  <xacro:include filename="$(find oslr)/urdf/oslr_navcam.xacro"/>
+  <xacro:include filename="$(find oslr_description)/urdf/oslr_base.xacro"/>
+  <xacro:include filename="$(find oslr_description)/urdf/oslr_rockerbogie.xacro"/>
+  <xacro:include filename="$(find oslr_description)/urdf/oslr_wheels.xacro"/>
+  <xacro:include filename="$(find oslr_description)/urdf/oslr_navcam.xacro"/>
   <!-- Load Gazebo plugin for ROS control -->
   <xacro:macro name="controller_plugin_gazebo" params="robot_namespace:=''">

File: oslr_description/urdf/oslr_base.xacro (robot description, xacro)
@@ -23,5 +23,6 @@
 #
 # References:
-#   ...
+#   References are listed in the README.
+#   Comments that include a [number] refers to the index in the reference list.
 #
 -->
@@ -62,5 +63,5 @@
       <geometry>
         <mesh
-          filename="package://oslr/models/oslr/meshes/base_link.STL" />
+          filename="package://oslr_description/models/oslr/meshes/base_link.STL" />
       </geometry>
       <material
@@ -76,5 +77,5 @@
       <geometry>
         <mesh
-          filename="package://oslr/models/oslr/meshes/base_link.STL" />
+          filename="package://oslr_description/models/oslr/meshes/base_link.STL" />
       </geometry>
     </collision>

File: oslr_description/urdf/oslr_navcam.xacro (robot description, xacro)
@@ -23,5 +23,6 @@
 #
 # References:
-#   ...
+#   References are listed in the README.
+#   Comments that include a [number] refers to the index in the reference list.
 #
 -->
@@ -38,4 +39,11 @@
   <xacro:property name="navcam_horiz_effort_lim" value="${yaml_dict['navcam_horiz_effort_lim']}" />
   <xacro:property name="navcam_horiz_velocity_lim" value="${yaml_dict['navcam_horiz_velocity_lim']}" />
+  <xacro:property name="navcam_baseline" value="${yaml_dict['navcam_baseline']}" />
+  <xacro:property name="navcam_update_rate" value="${yaml_dict['navcam_update_rate']}" />
+  <xacro:property name="navcam_fov" value="${yaml_dict['navcam_fov']}" />
+  <xacro:property name="navcam_image_width" value="${yaml_dict['navcam_image_width']}" />
+  <xacro:property name="navcam_image_height" value="${yaml_dict['navcam_image_height']}" />
+  <xacro:property name="navcam_clip_near" value="${yaml_dict['navcam_clip_near']}" />
+  <xacro:property name="navcam_clip_far" value="${yaml_dict['navcam_clip_far']}" />
   <xacro:property name="friction_coeff1_navcam_horiz" value="${yaml_dict['friction_coeff1_navcam_horiz']}" />
   <xacro:property name="friction_coeff2_navcam_horiz" value="${yaml_dict['friction_coeff2_navcam_horiz']}" />
@@ -69,5 +77,5 @@
       <geometry>
         <mesh
-          filename="package://oslr/models/oslr/meshes/navcam_horiz.STL" />
+          filename="package://oslr_description/models/oslr/meshes/navcam_horiz.STL" />
       </geometry>
       <material
@@ -83,5 +91,5 @@
       <geometry>
         <mesh
-          filename="package://oslr/models/oslr/meshes/navcam_horiz.STL" />
+          filename="package://oslr_description/models/oslr/meshes/navcam_horiz.STL" />
       </geometry>
     </collision>
@@ -127,5 +135,5 @@
       <geometry>
         <mesh
-          filename="package://oslr/models/oslr/meshes/navcam_vertical.STL" />
+          filename="package://oslr_description/models/oslr/meshes/navcam_vertical.STL" />
       </geometry>
       <material
@@ -141,5 +149,5 @@
       <geometry>
         <mesh
-          filename="package://oslr/models/oslr/meshes/navcam_vertical.STL" />
+          filename="package://oslr_description/models/oslr/meshes/navcam_vertical.STL" />
       </geometry>
     </collision>
@@ -185,5 +193,5 @@
       <geometry>
         <mesh
-          filename="package://oslr/models/oslr/meshes/navcam_eye_left.STL" />
+          filename="package://oslr_description/models/oslr/meshes/navcam_eye_left.STL" />
       </geometry>
       <material
@@ -199,5 +207,5 @@
       <geometry>
         <mesh
-          filename="package://oslr/models/oslr/meshes/navcam_eye_left.STL" />
+          filename="package://oslr_description/models/oslr/meshes/navcam_eye_left.STL" />
       </geometry>
     </collision>
@@ -238,5 +246,5 @@
       <geometry>
         <mesh
-          filename="package://oslr/models/oslr/meshes/navcam_eye_right.STL" />
+          filename="package://oslr_description/models/oslr/meshes/navcam_eye_right.STL" />
       </geometry>
       <material
@@ -252,5 +260,5 @@
       <geometry>
         <mesh
-          filename="package://oslr/models/oslr/meshes/navcam_eye_right.STL" />
+          filename="package://oslr_description/models/oslr/meshes/navcam_eye_right.STL" />
       </geometry>
     </collision>
@@ -300,5 +308,5 @@
   <gazebo reference="navcam_eye_left">
     <sensor type="multicamera" name="navcam">
-      <update_rate>15.0</update_rate>
+      <update_rate>${navcam_update_rate}</update_rate>
       <camera name="left">
         <!--
@@ -308,37 +316,37 @@
           +z                       | -y
         -->
-        <pose>0 0 0 0 -1.57 -1.57</pose>
-        <horizontal_fov>1.3962634</horizontal_fov>
+        <pose>0 0 0 0 ${-pi/2} ${-pi/2}</pose>
+        <horizontal_fov>${navcam_fov}</horizontal_fov>
         <image>
-          <width>400</width>
-          <height>400</height>
+          <width>${navcam_image_width}</width>
+          <height>${navcam_image_height}</height>
           <format>R8G8B8</format>
         </image>
         <clip>
-          <near>0.02</near>
-          <far>300</far>
+          <near>${navcam_clip_near}</near>
+          <far>${navcam_clip_far}</far>
         </clip>
         <noise>
           <type>gaussian</type>
           <mean>0.0</mean>
-          <stddev>0.007</stddev>
+          <stddev>0.0</stddev>
         </noise>
       </camera>
       <camera name="right">
-        <pose>-0.08 0 0 0 -1.57 -1.57</pose>
-        <horizontal_fov>1.3962634</horizontal_fov>
+        <pose>${-navcam_baseline} 0 0 0 ${-pi/2} ${-pi/2}</pose>
+        <horizontal_fov>${navcam_fov}</horizontal_fov>
         <image>
-          <width>400</width>
-          <height>400</height>
+          <width>${navcam_image_width}</width>
+          <height>${navcam_image_height}</height>
           <format>R8G8B8</format>
         </image>
         <clip>
-          <near>0.02</near>
-          <far>300</far>
+          <near>${navcam_clip_near}</near>
+          <far>${navcam_clip_far}</far>
         </clip>
         <noise>
           <type>gaussian</type>
           <mean>0.0</mean>
-          <stddev>0.007</stddev>
+          <stddev>0.0</stddev>
         </noise>
       </camera>
@@ -350,5 +358,5 @@
         <cameraInfoTopicName>camera_info</cameraInfoTopicName>
         <frameName>navcam_eye_left</frameName>
-        <hackBaseline>0.0</hackBaseline>
+        <hackBaseline>${navcam_baseline}</hackBaseline>
         <distortionK1>0.0</distortionK1>
         <distortionK2>0.0</distortionK2>

File: oslr_description/urdf/oslr_rockerbogie.xacro (robot description, xacro)
@@ -23,5 +23,6 @@
 #
 # References:
-#   ...
+#   References are listed in the README.
+#   Comments that include a [number] refers to the index in the reference list.
 #
 -->
@@ -86,5 +87,5 @@
       <geometry>
         <mesh
-          filename="package://oslr/models/oslr/meshes/left_rocker.STL" />
+          filename="package://oslr_description/models/oslr/meshes/left_rocker.STL" />
       </geometry>
       <material
@@ -100,5 +101,5 @@
       <geometry>
         <mesh
-          filename="package://oslr/models/oslr/meshes/left_rocker.STL" />
+          filename="package://oslr_description/models/oslr/meshes/left_rocker.STL" />
       </geometry>
     </collision>
@@ -148,5 +149,5 @@
       <geometry>
         <mesh
-          filename="package://oslr/models/oslr/meshes/left_bogie.STL" />
+          filename="package://oslr_description/models/oslr/meshes/left_bogie.STL" />
       </geometry>
       <material
@@ -162,5 +163,5 @@
       <geometry>
         <mesh
-          filename="package://oslr/models/oslr/meshes/left_bogie.STL" />
+          filename="package://oslr_description/models/oslr/meshes/left_bogie.STL" />
       </geometry>
     </collision>
@@ -206,5 +207,5 @@
       <geometry>
         <mesh
-          filename="package://oslr/models/oslr/meshes/right_rocker.STL" />
+          filename="package://oslr_description/models/oslr/meshes/right_rocker.STL" />
       </geometry>
       <material
@@ -220,5 +221,5 @@
       <geometry>
         <mesh
-          filename="package://oslr/models/oslr/meshes/right_rocker.STL" />
+          filename="package://oslr_description/models/oslr/meshes/right_rocker.STL" />
       </geometry>
     </collision>
@@ -264,5 +265,5 @@
       <geometry>
         <mesh
-          filename="package://oslr/models/oslr/meshes/right_bogie.STL" />
+          filename="package://oslr_description/models/oslr/meshes/right_bogie.STL" />
       </geometry>
       <material
@@ -278,5 +279,5 @@
       <geometry>
         <mesh
-          filename="package://oslr/models/oslr/meshes/right_bogie.STL" />
+          filename="package://oslr_description/models/oslr/meshes/right_bogie.STL" />
       </geometry>
     </collision>

File: oslr_description/urdf/oslr_wheels.xacro (robot description, xacro)
@@ -23,5 +23,6 @@
 #
 # References:
-#   ...
+#   References are listed in the README.
+#   Comments that include a [number] refers to the index in the reference list.
 #
 -->
@@ -44,4 +45,6 @@
   <xacro:property name="stiffness_corner" value="${yaml_dict['stiffness_corner']}" />
   <xacro:property name="damping_corner" value="${yaml_dict['damping_corner']}" />
+  <xacro:property name="steer_mech_reduction" value="${yaml_dict['steer_mech_reduction']}" />
+  <xacro:property name="drive_mech_reduction" value="${yaml_dict['drive_mech_reduction']}" />
   <!-- ********************************** GEOMETRY ********************************** -->
   <link
@@ -67,5 +70,5 @@
       <geometry>
         <mesh
-          filename="package://oslr/models/oslr/meshes/front_left_corner.STL" />
+          filename="package://oslr_description/models/oslr/meshes/front_left_corner.STL" />
       </geometry>
       <material
@@ -81,5 +84,5 @@
       <geometry>
         <mesh
-          filename="package://oslr/models/oslr/meshes/front_left_corner.STL" />
+          filename="package://oslr_description/models/oslr/meshes/front_left_corner.STL" />
       </geometry>
     </collision>
@@ -125,5 +128,5 @@
       <geometry>
         <mesh
-          filename="package://oslr/models/oslr/meshes/front_left_wheel.STL" />
+          filename="package://oslr_description/models/oslr/meshes/front_left_wheel.STL" />
       </geometry>
       <material
@@ -139,5 +142,5 @@
       <geometry>
         <mesh
-          filename="package://oslr/models/oslr/meshes/front_left_wheel.STL" />
+          filename="package://oslr_description/models/oslr/meshes/front_left_wheel.STL" />
       </geometry>
     </collision>
@@ -181,5 +184,5 @@
       <geometry>
         <mesh
-          filename="package://oslr/models/oslr/meshes/middle_left_wheel.STL" />
+          filename="package://oslr_description/models/oslr/meshes/middle_left_wheel.STL" />
       </geometry>
       <material
@@ -195,5 +198,5 @@
       <geometry>
         <mesh
-          filename="package://oslr/models/oslr/meshes/middle_left_wheel.STL" />
+          filename="package://oslr_description/models/oslr/meshes/middle_left_wheel.STL" />
       </geometry>
     </collision>
@@ -237,5 +240,5 @@
       <geometry>
         <mesh
-          filename="package://oslr/models/oslr/meshes/back_left_corner.STL" />
+          filename="package://oslr_description/models/oslr/meshes/back_left_corner.STL" />
       </geometry>
       <material
@@ -251,5 +254,5 @@
       <geometry>
         <mesh
-          filename="package://oslr/models/oslr/meshes/back_left_corner.STL" />
+          filename="package://oslr_description/models/oslr/meshes/back_left_corner.STL" />
       </geometry>
     </collision>
@@ -295,5 +298,5 @@
       <geometry>
         <mesh
-          filename="package://oslr/models/oslr/meshes/back_left_wheel.STL" />
+          filename="package://oslr_description/models/oslr/meshes/back_left_wheel.STL" />
       </geometry>
       <material
@@ -309,5 +312,5 @@
       <geometry>
         <mesh
-          filename="package://oslr/models/oslr/meshes/back_left_wheel.STL" />
+          filename="package://oslr_description/models/oslr/meshes/back_left_wheel.STL" />
       </geometry>
     </collision>
@@ -351,5 +354,5 @@
       <geometry>
         <mesh
-          filename="package://oslr/models/oslr/meshes/front_right_corner.STL" />
+          filename="package://oslr_description/models/oslr/meshes/front_right_corner.STL" />
       </geometry>
       <material
@@ -365,5 +368,5 @@
       <geometry>
         <mesh
-          filename="package://oslr/models/oslr/meshes/front_right_corner.STL" />
+          filename="package://oslr_description/models/oslr/meshes/front_right_corner.STL" />
       </geometry>
     </collision>
@@ -409,5 +412,5 @@
       <geometry>
         <mesh
-          filename="package://oslr/models/oslr/meshes/front_right_wheel.STL" />
+          filename="package://oslr_description/models/oslr/meshes/front_right_wheel.STL" />
       </geometry>
       <material
@@ -423,5 +426,5 @@
       <geometry>
         <mesh
-          filename="package://oslr/models/oslr/meshes/front_right_wheel.STL" />
+          filename="package://oslr_description/models/oslr/meshes/front_right_wheel.STL" />
       </geometry>
     </collision>
@@ -465,5 +468,5 @@
       <geometry>
         <mesh
-          filename="package://oslr/models/oslr/meshes/middle_right_wheel.STL" />
+          filename="package://oslr_description/models/oslr/meshes/middle_right_wheel.STL" />
       </geometry>
       <material
@@ -479,5 +482,5 @@
       <geometry>
         <mesh
-          filename="package://oslr/models/oslr/meshes/middle_right_wheel.STL" />
+          filename="package://oslr_description/models/oslr/meshes/middle_right_wheel.STL" />
       </geometry>
     </collision>
@@ -521,5 +524,5 @@
       <geometry>
         <mesh
-          filename="package://oslr/models/oslr/meshes/back_right_corner.STL" />
+          filename="package://oslr_description/models/oslr/meshes/back_right_corner.STL" />
       </geometry>
       <material
@@ -535,5 +538,5 @@
       <geometry>
         <mesh
-          filename="package://oslr/models/oslr/meshes/back_right_corner.STL" />
+          filename="package://oslr_description/models/oslr/meshes/back_right_corner.STL" />
       </geometry>
     </collision>
@@ -579,5 +582,5 @@
       <geometry>
         <mesh
-          filename="package://oslr/models/oslr/meshes/back_right_wheel.STL" />
+          filename="package://oslr_description/models/oslr/meshes/back_right_wheel.STL" />
       </geometry>
       <material
@@ -593,5 +596,5 @@
       <geometry>
         <mesh
-          filename="package://oslr/models/oslr/meshes/back_right_wheel.STL" />
+          filename="package://oslr_description/models/oslr/meshes/back_right_wheel.STL" />
       </geometry>
     </collision>
@@ -688,5 +691,5 @@
     <type>transmission_interface/SimpleTransmission</type>
     <actuator name="front_left_wheel_motor">
-      <mechanicalReduction>26.9</mechanicalReduction>
+      <mechanicalReduction>${drive_mech_reduction}</mechanicalReduction>
     </actuator>
     <joint name="front_left_drive_joint">
@@ -697,5 +700,5 @@
     <type>transmission_interface/SimpleTransmission</type>
     <actuator name="front_right_wheel_motor">
-      <mechanicalReduction>26.9</mechanicalReduction>
+      <mechanicalReduction>${drive_mech_reduction}</mechanicalReduction>
     </actuator>
     <joint name="front_right_drive_joint">
@@ -706,5 +709,5 @@
     <type>transmission_interface/SimpleTransmission</type>
     <actuator name="middle_left_wheel_motor">
-      <mechanicalReduction>26.9</mechanicalReduction>
+      <mechanicalReduction>${drive_mech_reduction}</mechanicalReduction>
     </actuator>
     <joint name="middle_left_drive_joint">
@@ -715,5 +718,5 @@
     <type>transmission_interface/SimpleTransmission</type>
     <actuator name="middle_right_wheel_motor">
-      <mechanicalReduction>26.9</mechanicalReduction>
+      <mechanicalReduction>${drive_mech_reduction}</mechanicalReduction>
     </actuator>
     <joint name="middle_right_drive_joint">
@@ -724,5 +727,5 @@
     <type>transmission_interface/SimpleTransmission</type>
     <actuator name="back_left_wheel_motor">
-      <mechanicalReduction>26.9</mechanicalReduction>
+      <mechanicalReduction>${drive_mech_reduction}</mechanicalReduction>
     </actuator>
     <joint name="back_left_drive_joint">
@@ -733,5 +736,5 @@
     <type>transmission_interface/SimpleTransmission</type>
     <actuator name="back_right_wheel_motor">
-      <mechanicalReduction>26.9</mechanicalReduction>
+      <mechanicalReduction>${drive_mech_reduction}</mechanicalReduction>
     </actuator>
     <joint name="back_right_drive_joint">
@@ -742,5 +745,5 @@
     <type>transmission_interface/SimpleTransmission</type>
     <actuator name="front_left_corner_motor">
-      <mechanicalReduction>189</mechanicalReduction>
+      <mechanicalReduction>${steer_mech_reduction}</mechanicalReduction>
     </actuator>
     <joint name="front_left_corner_joint">
@@ -751,5 +754,5 @@
     <type>transmission_interface/SimpleTransmission</type>
     <actuator name="front_right_corner_motor">
-      <mechanicalReduction>189</mechanicalReduction>
+      <mechanicalReduction>${steer_mech_reduction}</mechanicalReduction>
     </actuator>
     <joint name="front_right_corner_joint">
@@ -760,5 +763,5 @@
     <type>transmission_interface/SimpleTransmission</type>
     <actuator name="back_left_corner_motor">
-      <mechanicalReduction>189</mechanicalReduction>
+      <mechanicalReduction>${steer_mech_reduction}</mechanicalReduction>
     </actuator>
     <joint name="back_left_corner_joint">
@@ -769,5 +772,5 @@
     <type>transmission_interface/SimpleTransmission</type>
     <actuator name="back_right_corner_motor">
-      <mechanicalReduction>189</mechanicalReduction>
+      <mechanicalReduction>${steer_mech_reduction}</mechanicalReduction>
     </actuator>
     <joint name="back_right_corner_joint">
